File: GD32VF-Breakout.kicad_pcb (KiCad board)
At the start: 4 copper layers, 43.6 x 24.2 mm, 33 parts, among them J1 JTAG, J2 USB_Conn, J5 Conn_01x15, J6 Conn_01x15, SW1 BOOT0, SW2 Reset, U1 XC6206PxxxMR, U2 USBLC6-2SC6, U3 GD32VF103Tx, Y1 12MHz

Commit message: First changes
Parts:
- removed C1: 4u7, Capacitor_SMD:C_0603_1608Metric
- removed C10: 10n, Capacitor_SMD:C_0402_1005Metric
- removed C11, C12: 20p, Capacitor_SMD:C_0402_1005Metric
- removed C2, C3, C4, C7: 100n, Capacitor_SMD:C_0402_1005Metric
- removed C5, C6: 10u, Capacitor_SMD:C_0603_1608Metric
- removed C8: 4n7, Capacitor_SMD:C_0402_1005Metric
- removed C9: 1u, Capacitor_SMD:C_0603_1608Metric
- removed D1: Power, LED_SMD:LED_0603_1608Metric
- removed F1: 100mA, Fuse:Fuse_1206_3216Metric
- removed FB1: 100 @ 100MHz, Inductor_SMD:L_0805_2012Metric
- removed J1: JTAG, Connector_PinHeader_2.54mm:PinHeader_1x04_P2.54mm_Vertical
- removed J2: USB_Conn, Connector_USB:USB_C_Receptacle_HRO_TYPE-C-31-M-12
- removed J5, J6: Conn_01x15, Connector_PinHeader_2.54mm:PinHeader_1x15_P2.54mm_Vertical
- removed R1, R2, R7: 10k, Resistor_SMD:R_0402_1005Metric
- removed R3, R9: 1M, Resistor_SMD:R_0402_1005Metric
- removed R4: 2k2, Resistor_SMD:R_0402_1005Metric
- removed R5, R6: 5k5, Resistor_SMD:R_0402_1005Metric
- removed SW1: BOOT0, Button_Switch_SMD:SW_Push_1P1T_NO_CK_KMR2
- removed SW2: Reset, Button_Switch_SMD:SW_Push_1P1T_NO_CK_KMR2
- removed U1: XC6206PxxxMR, Package_TO_SOT_SMD:SOT-23-3
- removed U2: USBLC6-2SC6, Package_TO_SOT_SMD:SOT-23-6
- removed U3: GD32VF103Tx, Packages:QFN-36_EP_6x6_Pitch0.5mm
- removed Y1: 12MHz, Crystal:Crystal_SMD_3225-4Pin_3.2x2.5mm
- added C101: 4u7F, Capacitor_SMD:C_0603_1608Metric_Pad1.08x0.95mm_HandSolder, F.Cu at (133.1, 74.3)
- added C102: 100nF, Capacitor_SMD:C_0603_1608Metric_Pad1.08x0.95mm_HandSolder, F.Cu at (133.1, 75.8)
- added C103: 100nF, Capacitor_SMD:C_0603_1608Metric_Pad1.08x0.95mm_HandSolder, F.Cu at (140.6, 83.5)
- added C104: 100nF, Capacitor_SMD:C_0603_1608Metric_Pad1.08x0.95mm_HandSolder, F.Cu at (140.6, 77.5)
- added C105: 10uF, Capacitor_SMD:C_0603_1608Metric_Pad1.08x0.95mm_HandSolder, F.Cu at (157.9, 88.3)
- added C106: 6.8pF, Capacitor_SMD:C_0603_1608Metric_Pad1.08x0.95mm_HandSolder, F.Cu at (159.6, 88.3)
- added C107: 10uF, Capacitor_SMD:C_0603_1608Metric_Pad1.08x0.95mm_HandSolder, F.Cu at (152.9, 88.3)
- added C108: 100nF, Capacitor_SMD:C_0603_1608Metric_Pad1.08x0.95mm_HandSolder, F.Cu at (118.0, 61.3)
- added C109: 4n7F, Capacitor_SMD:C_0603_1608Metric_Pad1.08x0.95mm_HandSolder, F.Cu at (118.0, 63.8)
- added C110: 1uF, Capacitor_SMD:C_0603_1608Metric_Pad1.08x0.95mm_HandSolder, F.Cu at (118.0, 66.3)
- added C111: 10nF, Capacitor_SMD:C_0603_1608Metric_Pad1.08x0.95mm_HandSolder, F.Cu at (118.0, 68.8)
- added C112: 20pF, Capacitor_SMD:C_0603_1608Metric_Pad1.08x0.95mm_HandSolder, F.Cu at (128.3, 75.3)
- added C113: 20pF, Capacitor_SMD:C_0603_1608Metric_Pad1.08x0.95mm_HandSolder, F.Cu at (128.3, 81.0)
- added D101: Power, LED_SMD:LED_0603_1608Metric_Pad1.05x0.95mm_HandSolder, F.Cu at (150.6, 105.8)
- added FB101: 100 @ 100MHz, Inductor_SMD:L_1206_3216Metric_Pad1.22x1.90mm_HandSolder, F.Cu at (152.5, 93.0)
- added J101: USB_B_Micro, Connector_USB:USB_Micro-B_Amphenol_10118193-0001LF_Horizontal, F.Cu at (161.9, 80.5)
- added J102: JTAG, Connector_PinHeader_2.54mm:PinHeader_1x04_P2.54mm_Vertical, F.Cu at (120.4, 88.1)
- added J103: Conn_01x15, Connector_PinHeader_2.54mm:PinHeader_1x15_P2.54mm_Vertical, F.Cu at (104.5, 62.4)
- added J104: Conn_01x15, Connector_PinHeader_2.54mm:PinHeader_1x15_P2.54mm_Vertical, F.Cu at (109.1, 62.4)
- added L101: 2.2uH, Inductor_SMD_Extra:ANR6045, F.Cu at (158.0, 93.8)
- added R101: 10k, Resistor_SMD:R_0603_1608Metric_Pad0.98x0.95mm_HandSolder, F.Cu at (118.0, 76.4)
- added R102: 453k, Resistor_SMD:R_0603_1608Metric_Pad0.98x0.95mm_HandSolder, F.Cu at (155.5, 84.3)
- added R103: 2k2, Resistor_SMD:R_0603_1608Metric_Pad0.98x0.95mm_HandSolder, F.Cu at (148.9, 105.9)
- added R104: 100k, Resistor_SMD:R_0603_1608Metric_Pad0.98x0.95mm_HandSolder, F.Cu at (155.5, 85.8)
- added R105: 10k, Resistor_SMD:R_0603_1608Metric_Pad0.98x0.95mm_HandSolder, F.Cu at (122.3, 68.8)
- added R106: 1M, Resistor_SMD:R_0603_1608Metric_Pad0.98x0.95mm_HandSolder, F.Cu at (122.3, 71.3)
- added R107: 10k, Resistor_SMD:R_0603_1608Metric_Pad0.98x0.95mm_HandSolder, F.Cu at (138.2, 85.8)
- added R108: 1M, Resistor_SMD:R_0603_1608Metric_Pad0.98x0.95mm_HandSolder, F.Cu at (122.3, 76.4)
- added R109: 10k, Resistor_SMD:R_0603_1608Metric_Pad0.98x0.95mm_HandSolder, F.Cu at (126.7, 61.3)
- added R110: 10k, Resistor_SMD:R_0603_1608Metric_Pad0.98x0.95mm_HandSolder, F.Cu at (126.7, 63.8)
- added R111: 10k, Resistor_SMD:R_0603_1608Metric_Pad0.98x0.95mm_HandSolder, F.Cu at (126.7, 66.3)
- added R112: 10k, Resistor_SMD:R_0603_1608Metric_Pad0.98x0.95mm_HandSolder, F.Cu at (126.7, 68.8)
- added SW101: BOOT0, Button_Switch_SMD:SW_Push_1P1T_NO_CK_KMR2, F.Cu at (114.8, 88.1)
- added SW102: Reset, Button_Switch_SMD:SW_Push_1P1T_NO_CK_KMR2, F.Cu at (114.8, 92.8)
- added U101: TLV62569DRL, Package_TO_SOT_SMD:SOT-563, F.Cu at (155.3, 88.3)
- added U102: USBLC6-2SC6, Package_TO_SOT_SMD:SOT-23-6, F.Cu at (153.1, 80.8)
- added U103: GD32VF103Tx, Packages:QFN-36_EP_6x6_Pitch0.5mm, F.Cu at (136.3, 80.1)
- added Y101: 25MHz, Crystal:Crystal_SMD_3225-4Pin_3.2x2.5mm, F.Cu at (128.3, 78.2)
Routing:
- net (no net): track 0.00 -> 89.3 mm, vias 0 -> 2
- net +5V: track 66.0 -> 0.00 mm, vias 2 -> 0
- net Net-(J101-Shield): track 0.00 -> 11.6 mm
- net GND: track 57.7 -> 69.1 mm
- net +3.3V: track 33.2 -> 42.2 mm
- net OSC_IN: track 7.22 -> 16.2 mm
- net Net-(J2-SHIELD): track 7.26 -> 0.00 mm
- net OSC_OUT: track 5.04 -> 11.2 mm
- net Net-(U1-VI): track 5.26 -> 0.00 mm
- net Net-(U3-PB2): track 3.54 -> 0.00 mm
- net /FB: track 0.00 -> 3.49 mm
- net /BOOT1: track 0.00 -> 2.19 mm
- net Net-(F1-Pad2): track 1.98 -> 0.00 mm
- net Net-(J2-CC1): track 1.88 -> 0.00 mm
- net Net-(J2-CC2): track 1.79 -> 0.00 mm
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
Commit message: Full board, as sent for fabrication
Parts:
- removed C101: 4u7F, Capacitor_SMD:C_0603_1608Metric_Pad1.08x0.95mm_HandSolder
- removed C102, C103, C104, C108: 100nF, Capacitor_SMD:C_0603_1608Metric_Pad1.08x0.95mm_HandSolder
- removed C105, C107: 10uF, Capacitor_SMD:C_0603_1608Metric_Pad1.08x0.95mm_HandSolder
- removed C106: 6.8pF, Capacitor_SMD:C_0603_1608Metric_Pad1.08x0.95mm_HandSolder
- removed C109: 4n7F, Capacitor_SMD:C_0603_1608Metric_Pad1.08x0.95mm_HandSolder
- removed C110: 1uF, Capacitor_SMD:C_0603_1608Metric_Pad1.08x0.95mm_HandSolder
- removed C111: 10nF, Capacitor_SMD:C_0603_1608Metric_Pad1.08x0.95mm_HandSolder
- removed C112, C113: 20pF, Capacitor_SMD:C_0603_1608Metric_Pad1.08x0.95mm_HandSolder
- removed D101: Power, LED_SMD:LED_0603_1608Metric_Pad1.05x0.95mm_HandSolder
- removed FB101: 100 @ 100MHz, Inductor_SMD:L_1206_3216Metric_Pad1.22x1.90mm_HandSolder
- removed J101: USB_B_Micro, Connector_USB:USB_Micro-B_Amphenol_10118193-0001LF_Horizontal
- removed J102: JTAG, Connector_PinHeader_2.54mm:PinHeader_1x04_P2.54mm_Vertical
- removed J103, J104: Conn_01x15, Connector_PinHeader_2.54mm:PinHeader_1x15_P2.54mm_Vertical
- removed L101: 2.2uH, Inductor_SMD_Extra:ANR6045
- removed R101, R105, R107, R109, R110, R111, R112: 10k, Resistor_SMD:R_0603_1608Metric_Pad0.98x0.95mm_HandSolder
- removed R102: 453k, Resistor_SMD:R_0603_1608Metric_Pad0.98x0.95mm_HandSolder
- removed R103: 2k2, Resistor_SMD:R_0603_1608Metric_Pad0.98x0.95mm_HandSolder
- removed R104: 100k, Resistor_SMD:R_0603_1608Metric_Pad0.98x0.95mm_HandSolder
- removed R106, R108: 1M, Resistor_SMD:R_0603_1608Metric_Pad0.98x0.95mm_HandSolder
- removed SW101: BOOT0, Button_Switch_SMD:SW_Push_1P1T_NO_CK_KMR2
- removed SW102: Reset, Button_Switch_SMD:SW_Push_1P1T_NO_CK_KMR2
- removed U101: TLV62569DRL, Package_TO_SOT_SMD:SOT-563
- removed U102: USBLC6-2SC6, Package_TO_SOT_SMD:SOT-23-6
- removed U103: GD32VF103Tx, Packages:QFN-36_EP_6x6_Pitch0.5mm
- removed Y101: 25MHz, Crystal:Crystal_SMD_3225-4Pin_3.2x2.5mm
- added C1: 10uF, Capacitor_SMD:C_0603_1608Metric, F.Cu at (172.5, 102.7)
- added C10: 100nF, Capacitor_SMD:C_0402_1005Metric, F.Cu at (143.3, 93.3)
- added C11: 10nF, Capacitor_SMD:C_0402_1005Metric, F.Cu at (141.4, 101.0)
- added C12: 1uF, Capacitor_SMD:C_0603_1608Metric, F.Cu at (140.1, 101.4)
- added C13: 100nF, Capacitor_SMD:C_0402_1005Metric, F.Cu at (113.5, 91.2)
- added C14: 100nF, Capacitor_SMD:C_0402_1005Metric, F.Cu at (113.5, 89.2)
- added C15: 33pF, Capacitor_SMD:C_0603_1608Metric, F.Cu at (139.7, 93.1)
- added C16: 33pF, Capacitor_SMD:C_0603_1608Metric, F.Cu at (139.9, 98.8)
- added C3: 10uF, Capacitor_SMD:C_0603_1608Metric, F.Cu at (165.4, 102.7)
- added C4: 100nF, Capacitor_SMD:C_0603_1608Metric, F.Cu at (131.6, 101.1)
- added C5: 4n7F, Capacitor_SMD:C_0603_1608Metric, F.Cu at (172.0, 85.4)
- added C6: 4u7F, Capacitor_SMD:C_0603_1608Metric, F.Cu at (145.6, 90.9)
- added C7: 100nF, Capacitor_SMD:C_0402_1005Metric, F.Cu at (151.2, 103.7)
- added C8: 100nF, Capacitor_SMD:C_0402_1005Metric, F.Cu at (154.2, 95.2)
- added C9: 100nF, Capacitor_SMD:C_0402_1005Metric, F.Cu at (145.8, 92.2)
- added D1: Power, LED_SMD:LED_0805_2012Metric, F.Cu at (164.5, 108.0)
- added FB1: 100 @ 100MHz, Inductor_SMD:L_1206_3216Metric, F.Cu at (165.7, 96.3)
- added H1: MountingHole, MountingHole:MountingHole_2.2mm_M2, F.Cu at (113.0, 83.0)
- added H2: MountingHole, MountingHole:MountingHole_2.2mm_M2, F.Cu at (113.0, 111.0)
- added H3: MountingHole, MountingHole:MountingHole_2.2mm_M2, F.Cu at (173.0, 111.0)
- added J1: USB_B_Micro, Connector_USB:USB_Micro-B_Amphenol_10118193-0001LF_Horizontal, F.Cu at (174.6, 91.6)
- added J2: JTAG, Connector_PinHeader_2.54mm:PinHeader_1x04_P2.54mm_Vertical, F.Cu at (114.8, 105.6)
- added J3: Conn_01x15, Connector_PinHeader_2.54mm:PinHeader_1x15_P2.54mm_Vertical, F.Cu at (122.8, 111.4)
- added J4: Conn_01x15, Connector_PinHeader_2.54mm:PinHeader_1x15_P2.54mm_Vertical, F.Cu at (122.8, 82.6)
- added L1: 2.2uH, Inductor_SMD:L_1210_3225Metric, F.Cu at (171.1, 106.0)
- added R1: 10k, Resistor_SMD:R_0603_1608Metric, F.Cu at (118.7, 97.1)
- added R10: 10k, Resistor_SMD:R_0603_1608Metric, F.Cu at (118.7, 106.4)
- added R11: 10k, Resistor_SMD:R_0603_1608Metric, F.Cu at (151.2, 106.5)
- added R13: 4k7, Resistor_SMD:R_0402_1005Metric, F.Cu at (118.2, 92.6)
- added R14: 4k7, Resistor_SMD:R_0402_1005Metric, F.Cu at (118.2, 89.6)
- added R2: 10k, Resistor_SMD:R_0603_1608Metric, F.Cu at (120.8, 99.7)
- added R3: 10k, Resistor_SMD:R_0603_1608Metric, F.Cu at (118.7, 102.2)
- added R4: 10k, Resistor_SMD:R_0603_1608Metric, F.Cu at (133.1, 101.1)
- added R5: 453k, Resistor_SMD:R_0603_1608Metric, F.Cu at (168.9, 98.5)
- added R6: 2k2, Resistor_SMD:R_0603_1608Metric, F.Cu at (162.5, 108.2)
- added R7: 100k, Resistor_SMD:R_0603_1608Metric, F.Cu at (168.9, 100.3)
- added R8: 10k, Resistor_SMD:R_0603_1608Metric, F.Cu at (131.6, 95.6)
- added R9: 1M, Resistor_SMD:R_0603_1608Metric, F.Cu at (170.4, 85.4)
- added SW1: BOOT0, Button_Switch_SMD:SW_Push_1P1T_NO_CK_KMR2, F.Cu at (128.0, 95.5)
- added SW2: Reset, Button_Switch_SMD:SW_Push_1P1T_NO_CK_KMR2, F.Cu at (128.0, 101.1)
- added U1: TLV62569DRL, Package_TO_SOT_SMD:SOT-563, F.Cu at (168.9, 102.7)
- added U2: USBLC6-2SC6, Package_TO_SOT_SMD:SOT-23-6, F.Cu at (164.8, 91.9)
- added U3: GD32VF103Cx, Package_QFP:LQFP-48_7x7mm_P0.5mm, F.Cu at (148.5, 98.0)
- added U4: BME280, Package_LGA:Bosch_LGA-8_2.5x2.5mm_P0.65mm_ClockwisePinNumbering, F.Cu at (115.7, 90.5)
- added Y1: 16MHz, Crystal:Crystal_SMD_3225-4Pin_3.2x2.5mm, F.Cu at (139.8, 96.0)
Routing:
- net (no net): track 89.3 -> 0.00 mm, vias 2 -> 0
- net JTDO: track 0.00 -> 47.0 mm, vias 0 -> 2
- net JTDI: track 0.00 -> 46.8 mm, vias 0 -> 2
- net JTMS: track 0.00 -> 46.7 mm, vias 0 -> 2
- net JTCK: track 0.00 -> 45.9 mm, vias 0 -> 2
- net SCL: track 0.00 -> 38.1 mm, vias 0 -> 2
- net PA13: track 38.0 -> 0.00 mm, vias 1 -> 0
- net SDA: track 0.00 -> 36.2 mm, vias 0 -> 2
- net PB3: track 35.0 -> 0.00 mm, vias 1 -> 0
- net PA15: track 32.6 -> 0.00 mm, vias 1 -> 0
- net VBUS: track 1.67 -> 33.8 mm
- net PA14: track 31.9 -> 0.00 mm, vias 1 -> 0
- net GND: track 69.1 -> 41.9 mm, vias 21 -> 28
- net PB9: track 0.00 -> 25.9 mm
- net PB8: track 0.00 -> 24.3 mm
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- added copper zone on F.Cu, net +3.3V
- added copper zone on F.Cu, net /SW
- added copper zone on F.Cu, net /VIN
- added copper zone on F.Cu, net GND
Other:
- board size 43.6 x 24.2 mm -> 66 x 34 mm
- board text added: "+3V3"
- board text added: "GND"
- board text added: "PA0"
- board text added: "PA1"
- board text added: "PA2"
- board text added: "PA3"
- board text added: "PA4"
- board text added: "PA5"
- board text added: "PA6"
- board text added: "PA7"
- board text added: "PB0"
- board text added: "PB1"
- board text added: "PB10"
- board text added: "PB12"
- board text added: "PB13"
- board text added: "PB14"
- board text added: "PB3"
- board text added: "PB4"
- board text added: "PB5"
- board text added: "PB8"
- board text added: "PB9"
- board text added: "RESET"
- board text added: "VBUS"
- board text added: "X"
- board text added: "~{RST}"
- board text removed: "GD32VF-BOut"
- board text removed: "JLCJLCJLCJLC"
- board text removed: "RST"
