File: GD32VF-Breakout.kicad_sch (KiCad schematic)
At the start: 33 parts, among them J1 JTAG, J2 USB_Conn, J5 Conn_01x15, J6 Conn_01x15, SW1 BOOT0, SW2 Reset, U1 XC6206PxxxMR, U2 USBLC6-2SC6, U3 GD32VF103Tx, Y1 12MHz

Commit message: Added submodule for local libraries
Parts:
- U3: symbol GigaDeviceSemi:GD32VF103Tx -> GDSemi-local:GD32VF103Tx
Changed lines of the file:
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@@
 	)
 	(symbol
-		(lib_id "GigaDeviceSemi:GD32VF103Tx")
+		(lib_id "GDSemi-local:GD32VF103Tx")
 		(at 251.46 96.52 0)
 		(unit 1)
@@
 		)
 		(property "Footprint" "Packages:QFN-36_EP_6x6_Pitch0.5mm"
-			(at 246.38 106.68 0)
+			(at 248.412 135.89 0)
 			(effects
 				(font
@@
 		)
 		(property "Datasheet" "https://github.com/riscv-mcu/GD32VF103_DataSheets/blob/6607c559bd9a109a64227bdaac332bbb126cf24f/GD32VF103_Datasheet_Rev_1.0.pdf"
-			(at 246.38 106.68 0)
+			(at 247.904 131.826 0)
 			(effects
 				(font
@@
 		)
 		(property "Description" ""
-			(at 246.38 106.68 0)
+			(at 246.38 119.38 0)
 			(effects
 				(font

Commit message: First changes
Parts:
- removed F1: 100mA, Fuse:Fuse_1206_3216Metric, symbol Device:Fuse
- removed J2: USB_Conn, Connector_USB:USB_C_Receptacle_HRO_TYPE-C-31-M-12, symbol Connector:USB_C_Receptacle_USB2.0_14P
- removed R5, R6: 5k5, Resistor_SMD:R_0402_1005Metric, symbol Device:R_Small
- removed U1: XC6206PxxxMR, Package_TO_SOT_SMD:SOT-23-3, symbol Regulator_Linear:XC6206PxxxMR
- added C106: 6.8pF, Capacitor_SMD:C_0603_1608Metric_Pad1.08x0.95mm_HandSolder, symbol Device:C_Small
- added J101: USB_B_Micro, Connector_USB:USB_Micro-B_Amphenol_10118193-0001LF_Horizontal, symbol Connector:USB_B_Micro
- added L101: 2.2uH, Inductor_SMD_Extra:ANR6045, symbol Device:L_Small
- added R102: 453k, Resistor_SMD:R_0603_1608Metric_Pad0.98x0.95mm_HandSolder, symbol Device:R_Small
- added R104: 100k, Resistor_SMD:R_0603_1608Metric_Pad0.98x0.95mm_HandSolder, symbol Device:R_Small
- added R109, R110, R111, R112: 10k, Resistor_SMD:R_0603_1608Metric_Pad0.98x0.95mm_HandSolder, symbol Device:R_Small
- added U101: TLV62569DRL, Package_TO_SOT_SMD:SOT-563, symbol Regulator_Switching:TLV62569DRL
- C101: renamed from C1; value 4u7 -> 4u7F; footprint Capacitor_SMD:C_0603_1608Metric -> Capacitor_SMD:C_0603_1608Metric_Pad1.08x0.95mm_HandSolder
- C102: renamed from C2; value 100n -> 100nF; footprint Capacitor_SMD:C_0402_1005Metric -> Capacitor_SMD:C_0603_1608Metric_Pad1.08x0.95mm_HandSolder
- C103: renamed from C3; value 100n -> 100nF; footprint Capacitor_SMD:C_0402_1005Metric -> Capacitor_SMD:C_0603_1608Metric_Pad1.08x0.95mm_HandSolder
- C104: renamed from C4; value 100n -> 100nF; footprint Capacitor_SMD:C_0402_1005Metric -> Capacitor_SMD:C_0603_1608Metric_Pad1.08x0.95mm_HandSolder
- C105: renamed from C6; value 10u -> 10uF; footprint Capacitor_SMD:C_0603_1608Metric -> Capacitor_SMD:C_0603_1608Metric_Pad1.08x0.95mm_HandSolder
- C107: renamed from C5; value 10u -> 10uF; footprint Capacitor_SMD:C_0603_1608Metric -> Capacitor_SMD:C_0603_1608Metric_Pad1.08x0.95mm_HandSolder
- C108: renamed from C7; value 100n -> 100nF; footprint Capacitor_SMD:C_0402_1005Metric -> Capacitor_SMD:C_0603_1608Metric_Pad1.08x0.95mm_HandSolder
- C109: renamed from C8; value 4n7 -> 4n7F; footprint Capacitor_SMD:C_0402_1005Metric -> Capacitor_SMD:C_0603_1608Metric_Pad1.08x0.95mm_HandSolder; now not fitted
- C110: renamed from C9; value 1u -> 1uF; footprint Capacitor_SMD:C_0603_1608Metric -> Capacitor_SMD:C_0603_1608Metric_Pad1.08x0.95mm_HandSolder
- C111: renamed from C10; value 10n -> 10nF; footprint Capacitor_SMD:C_0402_1005Metric -> Capacitor_SMD:C_0603_1608Metric_Pad1.08x0.95mm_HandSolder
- C112: renamed from C11; value 20p -> 20pF; footprint Capacitor_SMD:C_0402_1005Metric -> Capacitor_SMD:C_0603_1608Metric_Pad1.08x0.95mm_HandSolder
- C113: renamed from C12; value 20p -> 20pF; footprint Capacitor_SMD:C_0402_1005Metric -> Capacitor_SMD:C_0603_1608Metric_Pad1.08x0.95mm_HandSolder
- D101: renamed from D1; footprint LED_SMD:LED_0603_1608Metric -> LED_SMD:LED_0603_1608Metric_Pad1.05x0.95mm_HandSolder
- FB101: renamed from FB1; footprint Inductor_SMD:L_0805_2012Metric -> Inductor_SMD:L_1206_3216Metric_Pad1.22x1.90mm_HandSolder
- R101: renamed from R1; footprint Resistor_SMD:R_0402_1005Metric -> Resistor_SMD:R_0603_1608Metric_Pad0.98x0.95mm_HandSolder
- R103: renamed from R4; footprint Resistor_SMD:R_0402_1005Metric -> Resistor_SMD:R_0603_1608Metric_Pad0.98x0.95mm_HandSolder
- R105: renamed from R2; footprint Resistor_SMD:R_0402_1005Metric -> Resistor_SMD:R_0603_1608Metric_Pad0.98x0.95mm_HandSolder
- R106: renamed from R3; footprint Resistor_SMD:R_0402_1005Metric -> Resistor_SMD:R_0603_1608Metric_Pad0.98x0.95mm_HandSolder; now not fitted
- R107: renamed from R7; footprint Resistor_SMD:R_0402_1005Metric -> Resistor_SMD:R_0603_1608Metric_Pad0.98x0.95mm_HandSolder
- R108: renamed from R9; footprint Resistor_SMD:R_0402_1005Metric -> Resistor_SMD:R_0603_1608Metric_Pad0.98x0.95mm_HandSolder
- Y101: renamed from Y1; value 12MHz -> 25MHz
- renumbered J1 to J102, J5 to J103, J6 to J104, SW1 to SW101, SW2 to SW102, U2 to U102, U3 to U103
Connections:
- net +5V is gone; now on net VBUS: J103.15 (Pin_15), J104.1 (Pin_1), U102.5 (VBUS)
- net +3.3V: now also C106.1, L101.2, R102.1, R110.1, R111.1, R112.1
- net GND: now also C106.2, J101.5 (GND), R104.2, R109.2, U101.2 (GND)
- net PA13: no longer J102.3 (Pin_3), U103.25 (PA13)
- net PA14: no longer J102.4 (Pin_4), U103.28 (PA14)
- net PA15: no longer J102.2 (Pin_2), U103.29 (PA15)
- net PB3: no longer J102.1 (Pin_1), U103.30 (PB3)
- net USB_CONN_D+: now also J101.3 (D+)
- net USB_CONN_D-: now also J101.2 (D-)
- net at C109.1, R106.2: now also J101.6 (Shield)
- net BOOT1: now reaches R107.1, U103.17 (PB2)
- net VIN: now reaches C107.1, FB101.2
- net VIN: now also U101.3 (VIN), U101.5 (EN)
- net VBUS: now reaches FB101.1
- net VBUS: now also J101.1 (VBUS)
- new net: L101.1, U101.4 (SW)
- new net FB: R102.2, R104.1, U101.1 (FB)
- new net JTCK: J102.4 (Pin_4), R109.1, U103.28 (PA14)
- new net JTDI: J102.2 (Pin_2), R111.2, U103.29 (PA15)
- new net JTDO: J102.1 (Pin_1), R110.2, U103.30 (PB3)
- new net JTMS: J102.3 (Pin_3), R112.2, U103.25 (PA13)
Other:
- moved on the sheet: C102, C103, C104, C105, C107, D101, FB101, R103

Commit message: Full board, as sent for fabrication
Parts:
- removed C106: 6.8pF, Capacitor_SMD:C_0603_1608Metric_Pad1.08x0.95mm_HandSolder, symbol Device:C_Small
- removed R107: 10k, Resistor_SMD:R_0603_1608Metric_Pad0.98x0.95mm_HandSolder, symbol Device:R_Small
- removed R108: 1M, Resistor_SMD:R_0603_1608Metric_Pad0.98x0.95mm_HandSolder, symbol Device:R_Small
- removed U103: GD32VF103Tx, Packages:QFN-36_EP_6x6_Pitch0.5mm, symbol GDSemi-local:GD32VF103Tx
- added C10, C13, C14: 100nF, Capacitor_SMD:C_0402_1005Metric, symbol Device:C_Small
- added H1, H2, H3: MountingHole, MountingHole:MountingHole_2.2mm_M2, symbol Mechanical:MountingHole
- added R11: 10k, Resistor_SMD:R_0603_1608Metric, symbol Device:R_Small
- added R13, R14: 4k7, Resistor_SMD:R_0402_1005Metric, symbol Device:R_Small
- added U3: GD32VF103Cx, Package_QFP:LQFP-48_7x7mm_P0.5mm, symbol GigaDeviceSemi:GD32VF103Cx
- added U4: BME280, Package_LGA:Bosch_LGA-8_2.5x2.5mm_P0.65mm_ClockwisePinNumbering, symbol Sensor:BME280
- C1: renamed from C105; footprint Capacitor_SMD:C_0603_1608Metric_Pad1.08x0.95mm_HandSolder -> Capacitor_SMD:C_0603_1608Metric
- C11: renamed from C111; footprint Capacitor_SMD:C_0603_1608Metric_Pad1.08x0.95mm_HandSolder -> Capacitor_SMD:C_0402_1005Metric
- C12: renamed from C110; footprint Capacitor_SMD:C_0603_1608Metric_Pad1.08x0.95mm_HandSolder -> Capacitor_SMD:C_0603_1608Metric
- C15: renamed from C112; value 20pF -> 33pF; footprint Capacitor_SMD:C_0603_1608Metric_Pad1.08x0.95mm_HandSolder -> Capacitor_SMD:C_0603_1608Metric
- C16: renamed from C113; value 20pF -> 33pF; footprint Capacitor_SMD:C_0603_1608Metric_Pad1.08x0.95mm_HandSolder -> Capacitor_SMD:C_0603_1608Metric
- C3: renamed from C107; footprint Capacitor_SMD:C_0603_1608Metric_Pad1.08x0.95mm_HandSolder -> Capacitor_SMD:C_0603_1608Metric
- C4: renamed from C108; footprint Capacitor_SMD:C_0603_1608Metric_Pad1.08x0.95mm_HandSolder -> Capacitor_SMD:C_0603_1608Metric
- C5: renamed from C109; footprint Capacitor_SMD:C_0603_1608Metric_Pad1.08x0.95mm_HandSolder -> Capacitor_SMD:C_0603_1608Metric
- C6: renamed from C101; footprint Capacitor_SMD:C_0603_1608Metric_Pad1.08x0.95mm_HandSolder -> Capacitor_SMD:C_0603_1608Metric
- C7: renamed from C102; footprint Capacitor_SMD:C_0603_1608Metric_Pad1.08x0.95mm_HandSolder -> Capacitor_SMD:C_0402_1005Metric
- C8: renamed from C103; footprint Capacitor_SMD:C_0603_1608Metric_Pad1.08x0.95mm_HandSolder -> Capacitor_SMD:C_0402_1005Metric
- C9: renamed from C104; footprint Capacitor_SMD:C_0603_1608Metric_Pad1.08x0.95mm_HandSolder -> Capacitor_SMD:C_0402_1005Metric
- D1: renamed from D101; footprint LED_SMD:LED_0603_1608Metric_Pad1.05x0.95mm_HandSolder -> LED_SMD:LED_0805_2012Metric
- FB1: renamed from FB101; footprint Inductor_SMD:L_1206_3216Metric_Pad1.22x1.90mm_HandSolder -> Inductor_SMD:L_1206_3216Metric
- L1: renamed from L101; footprint Inductor_SMD_Extra:ANR6045 -> Inductor_SMD:L_1210_3225Metric
- R1: renamed from R110; footprint Resistor_SMD:R_0603_1608Metric_Pad0.98x0.95mm_HandSolder -> Resistor_SMD:R_0603_1608Metric
- R10: renamed from R109; footprint Resistor_SMD:R_0603_1608Metric_Pad0.98x0.95mm_HandSolder -> Resistor_SMD:R_0603_1608Metric
- R2: renamed from R111; footprint Resistor_SMD:R_0603_1608Metric_Pad0.98x0.95mm_HandSolder -> Resistor_SMD:R_0603_1608Metric
- R3: renamed from R112; footprint Resistor_SMD:R_0603_1608Metric_Pad0.98x0.95mm_HandSolder -> Resistor_SMD:R_0603_1608Metric
- R4: renamed from R101; footprint Resistor_SMD:R_0603_1608Metric_Pad0.98x0.95mm_HandSolder -> Resistor_SMD:R_0603_1608Metric
- R5: renamed from R102; footprint Resistor_SMD:R_0603_1608Metric_Pad0.98x0.95mm_HandSolder -> Resistor_SMD:R_0603_1608Metric
- R6: renamed from R103; footprint Resistor_SMD:R_0603_1608Metric_Pad0.98x0.95mm_HandSolder -> Resistor_SMD:R_0603_1608Metric
- R7: renamed from R104; footprint Resistor_SMD:R_0603_1608Metric_Pad0.98x0.95mm_HandSolder -> Resistor_SMD:R_0603_1608Metric
- R8: renamed from R105; footprint Resistor_SMD:R_0603_1608Metric_Pad0.98x0.95mm_HandSolder -> Resistor_SMD:R_0603_1608Metric
- R9: renamed from R106; footprint Resistor_SMD:R_0603_1608Metric_Pad0.98x0.95mm_HandSolder -> Resistor_SMD:R_0603_1608Metric
- Y1: renamed from Y101; value 25MHz -> 16MHz
- renumbered J101 to J1, J102 to J2, J103 to J3, J104 to J4, SW101 to SW1, SW102 to SW2, U101 to U1, U102 to U2
Connections:
- net +3.3V: now also C10.1, C13.1, C14.1, R13.1, R14.2, U3.1 (VBAT), U3.24 (VDD_1), U3.36 (VDD_2), U3.48 (VDD_3), U3.9 (VDDA), U4.2 (CSB), U4.5 (SDO), U4.6 (VDDIO), U4.8 (VDD)
- net BOOT0: now also U3.44 (BOOT0)
- net BOOT1: now also R11.1, U3.20 (PB2)
- net GND: now also C10.2, C13.2, C14.2, R11.2, U3.23 (VSS_1), U3.35 (VSS_2), U3.47 (VSS_3), U3.8 (VSSA), U4.1 (GND), U4.7 (GND)
- net JTCK: now also J2.1 (Pin_1), U3.37 (PA14); no longer J2.4 (Pin_4)
- net JTDI: now also J2.3 (Pin_3), U3.38 (PA15); no longer J2.2 (Pin_2)
- net JTDO: now also J2.4 (Pin_4), U3.39 (PB3); no longer J2.1 (Pin_1)
- net JTMS: now also J2.2 (Pin_2), U3.34 (PA13); no longer J2.3 (Pin_3)
- net NRST: now also U3.7 (NRST)
- net OSC_IN: now also U3.5 (OSCIN)
- net OSC_OUT: now also U3.6 (OSCOUT)
- net PA0: now also U3.10 (PA0)
- net PA1: now also U3.11 (PA1)
- net PA10: now also U3.31 (PA10)
- net PA2: now also U3.12 (PA2)
- net PA3: now also U3.13 (PA3)
- net PA4: now also U3.14 (PA4)
- net PA5: now also U3.15 (PA5)
- net PA6: now also U3.16 (PA6)
- net PA7: now also U3.17 (PA7)
- net PA8: now also U3.29 (PA8)
- net PA9: now also U3.30 (PA9)
- net PB0: now also U3.18 (PB0)
- net PB1: now also U3.19 (PB1)
- net PB4: now also U3.40 (PB4)
- net PB5: now also U3.41 (PB5)
- net USB_D+: now also U3.33 (PA12)
- net USB_D-: now also U3.32 (PA11)
- net VBUS: no longer J4.1 (Pin_1)
- net SW: now reaches L1.1, U1.4 (SW)
- net PA13 renamed PB14
- net PB14: now also U3.27 (PB14)
- net PA14 renamed PB13
- net PB13: now also U3.26 (PB13)
- net PA15 renamed PB12
- net PB12: now also U3.25 (PB12)
- net PB6 renamed PB8
- net PB8: now also U3.45 (PB8)
- net PB7 renamed PB9
- net PB9: now also U3.46 (PB9)
- new net SCL: R13.2, U3.42 (PB6), U4.4 (SCK)
- new net SDA: R14.1, U3.43 (PB7), U4.3 (SDI)
- no-connect marks 0 -> 9
Other:
- moved on the sheet: C1, C11, C12, C15, C16, C3, C4, C5, C6, C7, C8, C9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
